File: damecan/damecan.kicad_pcb (KiCad board)
At the start: 2 copper layers, 40 x 32 mm, 9 parts, among them J1 UPDI_Socket, SW1 PWR_SWITCH, SW2 RotaryEncoder, SW3 REST_VAL, U1 ATtiny202-SS

Commit message: レビュー後の改善
Parts:
- J1: moved to F.Cu
Connections:
- net -BATT renamed GND
