File: damecan/damecan.kicad_sch (KiCad schematic)
At the start: 9 parts, among them J1 UPDI_Socket, SW1 PWR_SWITCH, SW2 RotaryEncoder, SW3 REST_VAL, U1 ATtiny202-SS

Commit message: レビュー後の改善
Connections:
- net -BATT renamed GND
Other:
- moved on the sheet: BT1, Module1, SW1
